File: PCB/keyboard.kicad_pcb (KiCad board)
At the start: 2 copper layers, 328.7 x 100.9 mm, 160 parts, among them J1 USB_mini_micro_B, U1 ATMEGA32U4, X1 Crystal_GND24_Small

Commit message: added standard 68 key layout
Parts:
- removed the REF** at (175.3, 76.2)
- removed the REF** at (364.7, 74.3)
- removed the REF** at (352.0, 75.4)
- removed the REF** at (352.7, 80.9)
- removed the REF** at (230.1, 40.0)
- removed the REF** at (379.0, 79.6)
- added D_R_ALT_STD_1: D, acheron_Components:D_SOD-123, B.Cu at (251.7, 132.6)
- added K_BCK_STD1: KEYSW, MX_Only:MXOnly-2U-NoLED, F.Cu at (307.2, 59.8)
- added K_CAPS_STD_2: KEYSW, MX_Only:MXOnly-1.75U-NoLED, F.Cu at (57.1, 97.9)
- added K_CMD_STD_1: KEYSW, MX_Only:MXOnly-1.25U-NoLED, F.Cu at (100.0, 136.0)
- added K_CMD_STD_3: KEYSW, MX_Only:MXOnly-1.25U-NoLED, F.Cu at (266.7, 136.0)
- added K_CTRL_STD_1: KEYSW, MX_Only:MXOnly-1.25U-NoLED, F.Cu at (52.4, 136.0)
- added K_MEN_STD_1: KEYSW, MX_Only:MXOnly-1.25U-NoLED, F.Cu at (290.5, 136.0)
- added K_R_ALT_STD_1: KEYSW, MX_Only:MXOnly-1.25U-NoLED, F.Cu at (242.9, 136.0)
- added K_SPACE_STD1: KEYSW, MX_Only:MXOnly-6.25U-NoLED, F.Cu at (171.5, 136.0)
- added K_WIN_STD_1: KEYSW, MX_Only:MXOnly-1.25U-NoLED, F.Cu at (76.2, 136.0)
- added REF**: via-0.6mm, usbc_footprint:via-0.6mm, F.Cu at (307.4, 68.3)
- added REF**: via-0.6mm, usbc_footprint:via-0.6mm, F.Cu at (285.0, 67.0)
- added REF**: via-0.6mm, usbc_footprint:via-0.6mm, F.Cu at (158.2, 88.4)
- added REF**: via-0.6mm, usbc_footprint:via-0.6mm, F.Cu at (347.6, 86.5)
- added REF**: via-0.6mm, usbc_footprint:via-0.6mm, F.Cu at (334.9, 87.6)
- added REF**: via-0.6mm, usbc_footprint:via-0.6mm, F.Cu at (335.6, 93.1)
- added REF**: via-0.6mm, usbc_footprint:via-0.6mm, F.Cu at (213.0, 52.2)
- added REF**: via-0.6mm, usbc_footprint:via-0.6mm, F.Cu at (361.9, 91.8)
- K_&lt;I1, K_&lt;I2, K_&lt;I3, K_CTRL1, K_TAB1: footprint MX_Alps_Hybrid:MX-1.5U-NoLED -> MX_Only:MXOnly-1.5U-NoLED
- K_&lt;I_E1, K_0, K_1, K_2, K_3, K_4, K_5, K_6, K_7, K_8, K_9, K_A1, K_B1, K_BSLSH1, K_C1, K_CBRAC1, K_COMMA1, K_D1, K_DELETE1, K_DOT1, K_DOWN1, K_E1, K_END1, K_EQUAL1, K_F1, K_FN1, K_G1, K_H1, K_HOME1, K_I1, K_INSERT1, K_J1, K_K1, K_L1, K_LEFT1, K_M1, K_MINUS1, K_N1, K_O1, K_OBRAC1, K_P1, K_Q1, K_QUOTE1, K_R1, K_RIGHT1, K_S1, K_SEMIC1, K_SLASH1, K_T1, K_U1, K_UP1, K_V1, K_W1, K_X1, K_Y1, K_Z1, K_`1: footprint MX_Alps_Hybrid:MX-1U-NoLED -> MX_Only:MXOnly-1U-NoLED
- K_ALT1, K_CAPS1, K_WIN1: footprint MX_Alps_Hybrid:MX-1.25U-NoLED -> MX_Only:MXOnly-1.25U-NoLED
- K_ENTER1, K_SHIFT2: footprint MX_Alps_Hybrid:MX-2.25U-NoLED -> MX_Only:MXOnly-2.25U-NoLED
- K_SHIFT1: footprint MX_Alps_Hybrid:MX-1.75U-NoLED -> MX_Only:MXOnly-1.75U-NoLED
- K_SPACE1: footprint MX_Alps_Hybrid:MX-7U-NoLED -> MX_Only:MXOnly-7U-NoLED
- moved D_SPACE1 38.0 mm to (178.7, 141.7)
- moved D_CAPS1 23.7 mm to (60.3, 101.1)
- moved D_BSLSH1 23.3 mm to (304.3, 62.8)
- moved D_O1 21.0 mm to (240.6, 81.6)
- moved K_0 21.0 mm to (240.5, 59.8)
- moved D_ALT1 21.0 mm to (306.0, 138.8)
- moved D_DOWN1 21.0 mm to (349.3, 138.8)
- moved D_LEFT1 21.0 mm to (330.4, 138.8)
- moved D_WIN1 21.0 mm to (93.3, 138.8)
- moved C1 21.0 mm to (338.6, 87.5)
- moved C2 21.0 mm to (347.6, 87.6)
- moved C3 21.0 mm to (332.0, 95.0)
- moved C4 21.0 mm to (351.6, 93.8)
- moved C5 21.0 mm to (338.0, 106.5)
- moved C8 21.0 mm to (331.1, 97.9)
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Routing:
- net col11: track 201.5 -> 239.8 mm
- net col7: track 279.5 -> 307.0 mm
- net col12: track 209.0 -> 227.4 mm
- net col13: track 165.4 -> 178.1 mm
- net col3: track 367.7 -> 379.2 mm
- net col2: track 368.2 -> 378.3 mm
- net Net-(D_BSLSH1-Pad2): track 11.4 -> 19.9 mm
- net Net-(D_R1-Pad2): track 19.7 -> 11.7 mm
- net Net-(D_SPACE1-Pad2): track 9.91 -> 17.5 mm
- net Net-(D_&lt;I2-Pad2): track 10.5 -> 17.7 mm
- net Net-(J1-Pad3): track 194.7 -> 188.2 mm
- net Net-(D_R_ALT_STD_1-Pad2): track 0.00 -> 6.27 mm
- net col14: track 117.4 -> 122.8 mm, vias 0 -> 1
- net col1: track 412.6 -> 417.5 mm
- net Net-(D_ALT1-Pad2): track 12.0 -> 16.8 mm
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
Commit message: added usb type c.
Parts:
- removed J1: USB_mini_micro_B, keyboard_parts:USB_miniB_hirose_5S8
- added ESD1: USBLC6-2SC6, Package_TO_SOT_SMD:SOT-23-6, B.Cu at (202.8, 106.3)
- added R5: 5.1k, Resistor_SMD:R_0805_2012Metric_Pad1.15x1.40mm_HandSolder, B.Cu at (204.9, 51.9)
- added R6: 5.1k, Resistor_SMD:R_0805_2012Metric_Pad1.15x1.40mm_HandSolder, B.Cu at (210.2, 52.8)
- added USB1: HRO-TYPE-C-31-M-12, usbc_footprint:HRO-TYPE-C-31-M-12, B.Cu at (207.3, 41.7)
Connections:
- R3 pad 2: Net-(J1-Pad2) -> /D-
- R4 pad 2: Net-(J1-Pad3) -> /D+
Routing:
- net Net-(J1-Pad2): track 200.5 -> 0.00 mm, vias 2 -> 0
- net Net-(J1-Pad3): track 188.2 -> 0.00 mm, vias 2 -> 0
- net /D-: track 0.00 -> 134.2 mm
- net /D+: track 0.00 -> 130.3 mm
- net /D+_esd_in: track 0.00 -> 65.9 mm, vias 0 -> 2
- net /D-_esd_in: track 0.00 -> 63.5 mm, vias 0 -> 2
- net VCC: track 237.2 -> 260.0 mm, vias 2 -> 5
- net Net-(J1-Pad6): track 11.8 -> 0.00 mm
- net row2: track 297.5 -> 303.0 mm, vias 2 -> 4
- net Net-(R6-Pad2): track 0.00 -> 3.43 mm
- net GND: track 8.36 -> 11.0 mm
- net Net-(R5-Pad2): track 0.00 -> 2.59 mm
- net Net-(D_8-Pad2): track 11.6 -> 11.8 mm, vias 0 -> 1
Other:
- board size 328.7 x 100.9 mm -> 328.7 x 102.2 mm
